File: logic/logic.sch (KiCad schematic (older format))
At the start: 5 parts, among them J0 COLS, J1 ROWS, J2 ISP-PROG-6, U0 ATSAMD21G18A-AUT, U1 BMA250E

Commit message: update logic board outline
Parts:
- J0, J1: footprint Pin_Headers:Pin_Header_Straight_1x15_Pitch1.27mm -> Connector_PinHeader_2.00mm:PinHeader_1x15_P2.00mm_Vertical
- J2: footprint Pin_Headers:Pin_Header_Straight_2x03_Pitch2.54mm -> Connector_PinHeader_2.54mm:PinHeader_2x03_P2.54mm_Vertical
- U1: footprint Housings_LGA:LGA-12_2x2mm_Pitch0.5mm -> Package_LGA:LGA-12_2x2mm_P0.5mm
Changed lines of the file:
@@
 EESchema Schematic File Version 4
+LIBS:logic-cache
 EELAYER 26 0
 EELAYER END
@@
 F 0 "J0" V 9767 1396 50  0000 C CNN
 F 1 "COLS" V 9676 1396 50  0000 C CNN
-F 2 "Pin_Headers:Pin_Header_Straight_1x15_Pitch1.27mm" H 9550 1400 50  0001 C CNN
+F 2 "Connector_PinHeader_2.00mm:PinHeader_1x15_P2.00mm_Vertical" H 9550 1400 50  0001 C CNN
 F 3 "~" H 9550 1400 50  0001 C CNN
 	1    9550 1400
@@
 F 0 "J1" H 8300 2250 50  0000 C CNN
 F 1 "ROWS" H 8300 3850 50  0000 C CNN
-F 2 "Pin_Headers:Pin_Header_Straight_1x15_Pitch1.27mm" H 8350 3050 50  0001 C CNN
+F 2 "Connector_PinHeader_2.00mm:PinHeader_1x15_P2.00mm_Vertical" H 8350 3050 50  0001 C CNN
 F 3 "~" H 8350 3050 50  0001 C CNN
 	1    8350 3050
@@
 F 0 "J2" H 6620 1596 50  0000 R CNN
 F 1 "ISP-PROG-6" H 6620 1505 50  0000 R CNN
-F 2 "Pin_Headers:Pin_Header_Straight_2x03_Pitch2.54mm" V 6650 1550 50  0001 C CNN
+F 2 "Connector_PinHeader_2.54mm:PinHeader_2x03_P2.54mm_Vertical" V 6650 1550 50  0001 C CNN
 F 3 " ~" H 5625 950 50  0001 C CNN
 	1    6900 1500
@@
 L Custom_Library:BMA250E U1
 U 1 1 5C22CD64
-P 8300 5650
-F 0 "U1" H 8350 6328 50  0000 C CNN
-F 1 "BMA250E" H 8350 6237 50  0000 C CNN
-F 2 "Housings_LGA:LGA-12_2x2mm_Pitch0.5mm" H 8450 6200 50  0001 L CNN
-F 3 "www.st.com/resource/en/datasheet/lis2hh12.pdf" H 7950 5650 50  0001 C CNN
-	1    8300 5650
+P 6550 5250
+F 0 "U1" H 6600 5928 50  0000 C CNN
+F 1 "BMA250E" H 6600 5837 50  0000 C CNN
+F 2 "Package_LGA:LGA-12_2x2mm_P0.5mm" H 6700 5800 50  0001 L CNN
+F 3 "www.st.com/resource/en/datasheet/lis2hh12.pdf" H 6200 5250 50  0001 C CNN
+	1    6550 5250
 	1    0    0    -1
 $EndComp

Commit message: Reassign pins to avoid crossing
Changed lines of the file:
@@
 Text GLabel 1950 5700 0    50   Input ~ 0
 RESET
-Text GLabel 3950 2700 2    50   Input ~ 0
+Text GLabel 1950 5500 0    50   Input ~ 0
 SWDIO
-Text GLabel 3950 2600 2    50   Input ~ 0
+Text GLabel 1950 5400 0    50   Input ~ 0
 SWCLK
 Text GLabel 1950 4000 0    50   Input ~ 0
@@
 Text GLabel 1950 2600 0    50   Input ~ 0
 COL_0
+Text GLabel 1950 5300 0    50   Input ~ 0
+ROW_7
+Text GLabel 1950 5200 0    50   Input ~ 0
+ROW_8
+Text GLabel 3950 3300 2    50   Input ~ 0
+ROW_9
+Text GLabel 3950 3200 2    50   Input ~ 0
+ROW_10
+Text GLabel 1950 5100 0    50   Input ~ 0
+ROW_11
+Text GLabel 1950 5000 0    50   Input ~ 0
+ROW_12
+Text GLabel 1950 4900 0    50   Input ~ 0
+ROW_13
 Text GLabel 1950 4800 0    50   Input ~ 0
-ROW_7
-Text GLabel 1950 4900 0    50   Input ~ 0
-ROW_8
-Text GLabel 1950 5000 0    50   Input ~ 0
-ROW_9
-Text GLabel 1950 5100 0    50   Input ~ 0
-ROW_10
-Text GLabel 1950 5200 0    50   Input ~ 0
-ROW_11
-Text GLabel 1950 5300 0    50   Input ~ 0
-ROW_12
-Text GLabel 1950 5400 0    50   Input ~ 0
-ROW_13
-Text GLabel 1950 5500 0    50   Input ~ 0
 ROW_14
 Text GLabel 1950 4700 0    50   Input ~ 0

Commit message: Add power net and route matrix connections
Connections:
- net labels added: +3.3V, GND
- wire segments 0 -> 8
Changed lines of the file:
@@
 U 1 1 5CC6E0C1
 P 2950 4200
-F 0 "U0" H 2950 2214 50  0000 C CNN
-F 1 "ATSAMD21G18A-AUT" H 2950 2123 50  0000 C CNN
+F 0 "U0" H 2200 5950 50  0000 C CNN
+F 1 "ATSAMD21G18A-AUT" H 4150 2550 50  0000 C CNN
 F 2 "Package_QFP:TQFP-48_7x7mm_P0.5mm" H 2000 2450 50  0001 C CNN
 F 3 "" H 2950 5200 50  0001 C CNN
@@
 	1    0    0    -1
 $EndComp
+$Comp
+L power:+3.3V #PWR?
+U 1 1 5CC6F763
+P 2950 2050
+F 0 "#PWR?" H 2950 1900 50  0001 C CNN
+F 1 "+3.3V" H 2965 2223 50  0000 C CNN
+F 2 "" H 2950 2050 50  0001 C CNN
+F 3 "" H 2950 2050 50  0001 C CNN
+	1    2950 2050
+	1    0    0    -1
+$EndComp
+$Comp
+L power:GND #PWR?
+U 1 1 5CC6F79D
+P 2950 6200
+F 0 "#PWR?" H 2950 5950 50  0001 C CNN
+F 1 "GND" H 2955 6027 50  0000 C CNN
+F 2 "" H 2950 6200 50  0001 C CNN
+F 3 "" H 2950 6200 50  0001 C CNN
+	1    2950 6200
+	1    0    0    -1
+$EndComp
+Wire Wire Line
+	2850 6100 2950 6100
+Wire Wire Line
+	2950 6100 2950 6200
+Wire Wire Line
+	3050 6100 2950 6100
+Connection ~ 2950 6100
+Wire Wire Line
+	2950 2050 2950 2300
+Wire Wire Line
+	2950 2300 2850 2300
+Connection ~ 2850 2300
+Wire Wire Line
+	2850 2300 2750 2300
+Wire Wire Line
+	3150 2300 3050 2300
+Connection ~ 2950 2300
+Connection ~ 3050 2300
+Wire Wire Line
+	3050 2300 2950 2300
+$Comp
+L power:+3.3V #PWR?
+U 1 1 5CC6F8F4
+P 6800 1000
+F 0 "#PWR?" H 6800 850 50  0001 C CNN
+F 1 "+3.3V" H 6815 1173 50  0000 C CNN
+F 2 "" H 6800 1000 50  0001 C CNN
+F 3 "" H 6800 1000 50  0001 C CNN
+	1    6800 1000
+	1    0    0    -1
+$EndComp
+$Comp
+L power:GND #PWR?
+U 1 1 5CC6F90E
+P 6800 1900
+F 0 "#PWR?" H 6800 1650 50  0001 C CNN
+F 1 "GND" H 6805 1727 50  0000 C CNN
+F 2 "" H 6800 1900 50  0001 C CNN
+F 3 "" H 6800 1900 50  0001 C CNN
+	1    6800 1900
+	1    0    0    -1
+$EndComp
