File: dial/dial.sch (KiCad schematic (older format))
At the start: 65 parts, among them U1 MAX6951

Commit message: add components
Parts:
- added BT1: Battery_Cell, Custom Footprints:3008_coin_cell, symbol Device:Battery_Cell
- added C1, C2, C3, C4, C5: C_Small, Capacitor_SMD:C_0402_1005Metric, symbol Device:C_Small
- added SW1, SW2, SW3: SW_Push, Button_Switch_SMD:Panasonic_EVQPUK_EVQPUB, symbol Custom_Library:SW_Push
- added U2: ATSAMD10C14A-SS, Package_SO:SOIC-14_3.9x8.7mm_P1.27mm, symbol MCU_Microchip_SAMD:ATSAMD10C14A-SS
- added U3: BMA250E, Package_LGA:LGA-12_2x2mm_P0.5mm, symbol Custom_Library:BMA250E
- added Y1: Crystal_Small, Crystal:Crystal_SMD_5032-2Pin_5.0x3.2mm, symbol Device:Crystal_Small
Changed lines of the file:
@@
 EESchema Schematic File Version 4
+LIBS:dial-cache
 EELAYER 29 0
 EELAYER END
@@
 Text GLabel 3200 3150 3    50   Input ~ 0
 SEG3
+$Comp
+L MCU_Microchip_SAMD:ATSAMD10C14A-SS U2
+U 1 1 5CD3709A
+P 9400 2500
+F 0 "U2" H 9400 3381 50  0000 C CNN
+F 1 "ATSAMD10C14A-SS" H 9400 3290 50  0000 C CNN
+F 2 "Package_SO:SOIC-14_3.9x8.7mm_P1.27mm" H 9400 1450 50  0001 C CNN
+F 3 "" H 9400 1800 50  0001 C CNN
+	1    9400 2500
+	1    0    0    -1
+$EndComp
+$Comp
+L Device:Crystal_Small Y1
+U 1 1 5CD383F9
+P 11050 1900
+F 0 "Y1" H 11050 2125 50  0000 C CNN
+F 1 "Crystal_Small" H 11050 2034 50  0000 C CNN
+F 2 "Crystal:Crystal_SMD_5032-2Pin_5.0x3.2mm" H 11050 1900 50  0001 C CNN
+F 3 "~" H 11050 1900 50  0001 C CNN
+	1    11050 1900
+	1    0    0    -1
+$EndComp
+$Comp
+L Device:C_Small C4
+U 1 1 5CD3A587
+P 11350 2200
+F 0 "C4" H 11442 2246 50  0000 L CNN
+F 1 "C_Small" H 11442 2155 50  0000 L CNN
+F 2 "Capacitor_SMD:C_0402_1005Metric" H 11350 2200 50  0001 C CNN
+F 3 "~" H 11350 2200 50  0001 C CNN
+	1    11350 2200
+	1    0    0    -1
+$EndComp
+$Comp
+L Custom_Library:SW_Push SW2
+U 1 1 5CD410BE
+P 7550 2250
+F 0 "SW2" H 7550 2535 50  0000 C CNN
+F 1 "SW_Push" H 7550 2444 50  0000 C CNN
+F 2 "Button_Switch_SMD:Panasonic_EVQPUK_EVQPUB" H 7550 2450 50  0001 C CNN
+F 3 "" H 7550 2450 50  0001 C CNN
+	1    7550 2250
+	1    0    0    -1
+$EndComp
+$Comp
+L Custom_Library:BMA250E U3
+U 1 1 5CD42B85
+P 13150 3350
+F 0 "U3" H 13200 4031 50  0000 C CNN
+F 1 "BMA250E" H 13200 3940 50  0000 C CNN
+F 2 "Package_LGA:LGA-12_2x2mm_P0.5mm" H 13300 3900 50  0001 L CNN
+F 3 "" H 12800 3350 50  0001 C CNN
+	1    13150 3350
+	1    0    0    -1
+$EndComp
+$Comp
+L Device:Battery_Cell BT1
+U 1 1 5CD554BB
+P 7650 4050
+F 0 "BT1" H 7768 4146 50  0000 L CNN
+F 1 "Battery_Cell" H 7768 4055 50  0000 L CNN
+F 2 "Custom Footprints:3008_coin_cell" V 7650 4110 50  0001 C CNN
+F 3 "~" V 7650 4110 50  0001 C CNN
+	1    7650 4050
+	1    0    0    -1
+$EndComp
+$Comp
+L Device:C_Small C3
+U 1 1 5CD5928E
+P 10750 2200
+F 0 "C3" H 10842 2246 50  0000 L CNN
+F 1 "C_Small" H 10842 2155 50  0000 L CNN
+F 2 "Capacitor_SMD:C_0402_1005Metric" H 10750 2200 50  0001 C CNN
+F 3 "~" H 10750 2200 50  0001 C CNN
+	1    10750 2200
+	1    0    0    -1
+$EndComp
+$Comp
+L Custom_Library:SW_Push SW3
+U 1 1 5CD59951
+P 7600 2750
+F 0 "SW3" H 7600 3035 50  0000 C CNN
+F 1 "SW_Push" H 7600 2944 50  0000 C CNN
+F 2 "Button_Switch_SMD:Panasonic_EVQPUK_EVQPUB" H 7600 2950 50  0001 C CNN
+F 3 "" H 7600 2950 50  0001 C CNN
+	1    7600 2750
+	1    0    0    -1
+$EndComp
+$Comp
+L Custom_Library:SW_Push SW1
+U 1 1 5CD5A208
+P 7550 1750
+F 0 "SW1" H 7550 2035 50  0000 C CNN
+F 1 "SW_Push" H 7550 1944 50  0000 C CNN
+F 2 "Button_Switch_SMD:Panasonic_EVQPUK_EVQPUB" H 7550 1950 50  0001 C CNN
+F 3 "" H 7550 1950 50  0001 C CNN
+	1    7550 1750
+	1    0    0    -1
+$EndComp
+$Comp
+L Device:C_Small C2
+U 1 1 5CD5A96D
+P 10000 1750
+F 0 "C2" H 10092 1796 50  0000 L CNN
+F 1 "C_Small" H 10092 1705 50  0000 L CNN
+F 2 "Capacitor_SMD:C_0402_1005Metric" H 10000 1750 50  0001 C CNN
+F 3 "~" H 10000 1750 50  0001 C CNN
+	1    10000 1750
+	1    0    0    -1
+$EndComp
+$Comp
+L Device:C_Small C1
+U 1 1 5CD5B103
+P 9700 4900
+F 0 "C1" H 9792 4946 50  0000 L CNN
+F 1 "C_Small" H 9792 4855 50  0000 L CNN
+F 2 "Capacitor_SMD:C_0402_1005Metric" H 9700 4900 50  0001 C CNN
+F 3 "~" H 9700 4900 50  0001 C CNN
+	1    9700 4900
+	1    0    0    -1
+$EndComp
+$Comp
+L Device:C_Small C5
+U 1 1 5CD5B908
+P 13700 2700
+F 0 "C5" H 13792 2746 50  0000 L CNN
+F 1 "C_Small" H 13792 2655 50  0000 L CNN
+F 2 "Capacitor_SMD:C_0402_1005Metric" H 13700 2700 50  0001 C CNN
+F 3 "~" H 13700 2700 50  0001 C CNN
+	1    13700 2700
+	1    0    0    -1
+$EndComp
 $EndSCHEMATC
