File: dial/dial.sch (KiCad schematic (older format))
At the start: 77 parts, among them J1 SWD-PROG-6, SW1 UP, SW2 OK, SW3 DOWN, U0 ATSAMD21G18A-AUT, U1 BMA250E, Y1 32.768KHz

Commit message: Wired it all up
Parts:
- removed BT1: Battery_Cell, Battery:BatteryHolder_Keystone_3002_1x2032, symbol Device:Battery_Cell
- added C4, C5, C6: 1uF, Capacitor_SMD:C_0402_1005Metric, symbol Device:C
- added C7, C8: 4.7uF, Capacitor_SMD:C_0402_1005Metric, symbol Device:C
- added J0: Battery Pads, Custom Footprints:150mAh-Lipo, symbol Connector_Generic:Conn_01x02
- added R5, R6: 10M, Resistor_SMD:R_0402_1005Metric, symbol Device:R
- added R7: 2K, Resistor_SMD:R_0402_1005Metric, symbol Device:R
- added U2: Reg, Package_TO_SOT_SMD:SOT-23, symbol Regulator_Linear:APE8865N-33-HF-3
- added U3: CHG CTRL, Package_TO_SOT_SMD:SOT-23-5, symbol Battery_Management:MCP73831-2-OT
Connections:
- net +BATT: now also C4.1, C7.1, J0.1 (Pin_1), R5.1, U2.3 (VI), U3.3 (VBAT); no longer C0.2, C1.1, J1.2 (VCC), U0.17 (VDDIO), U0.36 (VDDIO), U0.43 (VDDCORE), U0.44 (VDDIN), U0.6 (VDDANA), U1.3 (VddIO), U1.7 (Vdd)
- net GND: now also U1.11 (PS), U1.5 (INT1), U1.6 (INT2), C4.2, C5.2, C6.2, C7.2, C8.2, J0.2 (Pin_2), R6.2, R7.2, U2.1 (GND), U3.2 (VSS)
- net SDO: now reaches U1.1 (SDO)
- net SDO: now also U0.29 (PA20)
- net CSB: now reaches U1.10 (~CSB)
- net CSB: now also U0.31 (PA22)
- net SCx: now reaches U1.12 (SCx)
- net SCx: now also U0.30 (PA21)
- net SDx: now reaches U1.2 (SDx)
- net SDx: now also U0.28 (PA19)
- net BAT_MON: now reaches U0.8 (PB09)
- net BAT_MON: now also C6.1, R5.2, R6.1
- new net: R7.1, U3.5 (PROG)
- new net +3V3: C0.2, C1.1, C5.1, U0.17 (VDDIO), U0.36 (VDDIO), U0.43 (VDDCORE), U0.44 (VDDIN), U0.6 (VDDANA), U1.3 (VddIO), U1.7 (Vdd), U2.2 (VO)
- new net CHARGE: C8.1, J1.2 (VCC), U3.4 (VDD)
Other:
- moved on the sheet: C0, C2, C3, R0, R1, R2, R3, R4, SW1, SW2, SW3, U0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
