File: Spark.sch (KiCad schematic (older format))
At the start: 87 parts, among them J0 Battery Pads, J1 SWD-PROG-6, SW1 UP, SW2 OK, SW3 DOWN, U0 ATSAMD21G18A-AUT, U1 BMA250E, U2 Reg, U3 CHG CTRL, Y1 32.768KHz

Commit message: initial rework to atmega1284p
Parts:
- removed C4, C5, C6: 1uF, Capacitor_SMD:C_0402_1005Metric, symbol Device:C
- removed C7, C8: 4.7uF, Capacitor_SMD:C_0805_2012Metric, symbol Device:C
- removed J1: SWD-PROG-6, Custom Footprints:ISP_SMD, symbol Custom_Library:SWD-PROG-6
- removed R5, R6: 10M, Resistor_SMD:R_0402_1005Metric, symbol Device:R
- removed R7: 2K, Resistor_SMD:R_0805_2012Metric, symbol Device:R
- removed U0: ATSAMD21G18A-AUT, Package_QFP:TQFP-48_7x7mm_P0.5mm, symbol MCU_Microchip_SAMD:ATSAMD21G18A-AUT
- removed U2: Reg, Package_TO_SOT_SMD:SOT-23, symbol Regulator_Linear:APE8865N-33-HF-3
- removed U3: CHG CTRL, Package_TO_SOT_SMD:SOT-23-5, symbol Battery_Management:MCP73831-2-OT
- added J1: ISP-PROG-6, Custom_Footprints:ISP_SMD, symbol Custom_Library:ISP-PROG-6
- added U0: ATmega1284P-AU, Package_QFP:TQFP-44_10x10mm_P0.8mm, symbol MCU_Microchip_ATmega:ATmega1284P-AU
- J0: footprint Custom Footprints:150mAh-Lipo -> Custom_Footprints:2-pin-SMD
- U1: value BMA250E -> BMA280
- Y1: footprint Crystal:Crystal_SMD_5032-2Pin_5.0x3.2mm -> Crystal:Crystal_SMD_3215-2Pin_3.2x1.5mm
Connections:
- net labels added: ACC_INT, CS, MISO, MOSI, SCK, TOSC1, TOSC2
- net labels removed: +3.3V, CHARGE, CSB, SCx, SDO, SDx, SWCLK, SWDIO, XIN, XOUT
- wire segments 121 -> 93
- no-connect marks 0 -> 2
Other:
- moved on the sheet: C0, R0, R1, R2, R3, R4, SW1, SW2, SW3

Commit message: erm, well, I did this ages ago so...
Parts:
- J0: footprint Custom_Footprints:2-pin-SMD -> Battery:BatteryHolder_Keystone_3002_1x2032
Connections:
- net EIGHT: now also U0.41 (PB1); no longer U0.16 (PD7)
- net ELEVEN: now also U0.22 (PC3); no longer U0.21 (PC2)
- net FIVE: now also U0.11 (PD2); no longer U0.13 (PD4)
- net NINE: now also U0.33 (PA4); no longer U0.19 (PC0)
- net ONE: now also U0.20 (PC1); no longer U0.9 (PD0)
- net SEVEN: now also U0.42 (PB2); no longer U0.15 (PD6)
- net SIX: now also U0.43 (PB3); no longer U0.14 (PD5)
- net TEN: now also U0.32 (PA5); no longer U0.20 (PC1)
- net THREE: now also U0.14 (PD5); no longer U0.11 (PD2)
- net TWELVE: now also U0.21 (PC2); no longer U0.22 (PC3)
- net TWO: now also U0.19 (PC0); no longer U0.10 (PD1)
- net at SW2.2: now also U0.13 (PD4); no longer U0.43 (PB3)
- net at SW3.2: now also U0.15 (PD6); no longer U0.42 (PB2)
- net at SW1.2: now also U0.16 (PD7); no longer U0.41 (PB1)
Other:
- moved on the sheet: J0, SW1, SW2, SW3
Changed lines of the file:
@@
 L Custom_Library:SW_Push SW2
 U 1 1 5CD410BE
-P 10700 3800
-F 0 "SW2" H 10700 4085 50  0000 C CNN
-F 1 "OK" H 10700 3994 50  0000 C CNN
-F 2 "Button_Switch_SMD:Panasonic_EVQPUK_EVQPUB" H 10700 4000 50  0001 C CNN
-F 3 "" H 10700 4000 50  0001 C CNN
-	1    10700 3800
+P 10700 5700
+F 0 "SW2" H 10700 5985 50  0000 C CNN
+F 1 "OK" H 10700 5894 50  0000 C CNN
+F 2 "Button_Switch_SMD:Panasonic_EVQPUK_EVQPUB" H 10700 5900 50  0001 C CNN
+F 3 "" H 10700 5900 50  0001 C CNN
+	1    10700 5700
 	-1   0    0    1
 $EndComp
@@
 L Custom_Library:SW_Push SW3
 U 1 1 5CD59951
-P 10700 3700
-F 0 "SW3" H 10700 3985 50  0000 C CNN
-F 1 "DOWN" H 10700 3894 50  0000 C CNN
-F 2 "Button_Switch_SMD:Panasonic_EVQPUK_EVQPUB" H 10700 3900 50  0001 C CNN
-F 3 "" H 10700 3900 50  0001 C CNN
-	1    10700 3700
+P 10700 5900
+F 0 "SW3" H 10700 6185 50  0000 C CNN
+F 1 "DOWN" H 10700 6094 50  0000 C CNN
+F 2 "Button_Switch_SMD:Panasonic_EVQPUK_EVQPUB" H 10700 6100 50  0001 C CNN
+F 3 "" H 10700 6100 50  0001 C CNN
+	1    10700 5900
 	-1   0    0    1
 $EndComp
@@
 L Custom_Library:SW_Push SW1
 U 1 1 5CD5A208
-P 10700 3600
-F 0 "SW1" H 10700 3885 50  0000 C CNN
-F 1 "UP" H 10700 3794 50  0000 C CNN
-F 2 "Button_Switch_SMD:Panasonic_EVQPUK_EVQPUB" H 10700 3800 50  0001 C CNN
-F 3 "" H 10700 3800 50  0001 C CNN
-	1    10700 3600
+P 10700 6000
+F 0 "SW1" H 10700 6285 50  0000 C CNN
+F 1 "UP" H 10700 6194 50  0000 C CNN
+F 2 "Button_Switch_SMD:Panasonic_EVQPUK_EVQPUB" H 10700 6200 50  0001 C CNN
+F 3 "" H 10700 6200 50  0001 C CNN
+	1    10700 6000
 	-1   0    0    1
 $EndComp
@@
 	0    -1   -1   0
 $EndComp
+Text GLabel 10500 4700 2    50   Input ~ 0
+ELEVEN
 Text GLabel 10500 4600 2    50   Input ~ 0
-ELEVEN
-Text GLabel 10500 4700 2    50   Input ~ 0
 TWELVE
-Text GLabel 10500 5300 2    50   Input ~ 0
+Text GLabel 10500 4500 2    50   Input ~ 0
 ONE
-Text GLabel 10500 5400 2    50   Input ~ 0
+Text GLabel 10500 4400 2    50   Input ~ 0
 TWO
-Text GLabel 10500 5500 2    50   Input ~ 0
+Text GLabel 10500 5800 2    50   Input ~ 0
 THREE
 Text GLabel 10500 5600 2    50   Input ~ 0
 FOUR
-Text GLabel 10500 5700 2    50   Input ~ 0
+Text GLabel 10500 5500 2    50   Input ~ 0
 FIVE
-Text GLabel 10500 5800 2    50   Input ~ 0
+Text GLabel 10500 3800 2    50   Input ~ 0
 SIX
-Text GLabel 10500 5900 2    50   Input ~ 0
+Text GLabel 10500 3700 2    50   Input ~ 0
 SEVEN
-Text GLabel 10500 6000 2    50   Input ~ 0
+Text GLabel 10500 3600 2    50   Input ~ 0
 EIGHT
-Text GLabel 10500 4400 2    50   Input ~ 0
+Text GLabel 10500 3000 2    50   Input ~ 0
 NINE
-Text GLabel 10500 4500 2    50   Input ~ 0
+Text GLabel 10500 3100 2    50   Input ~ 0
 TEN
 $Comp
 L power:GND #PWR0110
 U 1 1 5DFD6931
-P 11100 3900
-F 0 "#PWR0110" H 11100 3650 50  0001 C CNN
-F 1 "GND" H 11105 3727 50  0000 C CNN
-F 2 "" H 11100 3900 50  0001 C CNN
-F 3 "" H 11100 3900 50  0001 C CNN
-	1    11100 3900
-	1    0    0    -1
-$EndComp
-Wire Wire Line
-	10900 3800 11100 3800
-Wire Wire Line
-	11100 3800 11100 3900
-Connection ~ 10900 3800
-Wire Wire Line
-	10900 3700 10900 3800
+P 12400 4750
+F 0 "#PWR0110" H 12400 4500 50  0001 C CNN
+F 1 "GND" H 12405 4577 50  0000 C CNN
+F 2 "" H 12400 4750 50  0001 C CNN
+F 3 "" H 12400 4750 50  0001 C CNN
+	1    12400 4750
+	1    0    0    -1
+$EndComp
+Wire Wire Line
+	12200 4650 12400 4650
+Wire Wire Line
+	12400 4650 12400 4750
 $Comp
 L power:GND #PWR0111
@@
 L Connector_Generic:Conn_01x02 J0
 U 1 1 5D67BC28
-P 15300 7850
-F 0 "J0" V 15173 7930 50  0000 L CNN
-F 1 "Battery Pads" V 15264 7930 50  0000 L CNN
-F 2 "Custom_Footprints:2-pin-SMD" H 15300 7850 50  0001 C CNN
-F 3 "~" H 15300 7850 50  0001 C CNN
-	1    15300 7850
+P 13250 5200
+F 0 "J0" V 13123 5280 50  0000 L CNN
+F 1 "Battery Pads" V 13214 5280 50  0000 L CNN
+F 2 "Battery:BatteryHolder_Keystone_3002_1x2032" H 13250 5200 50  0001 C CNN
+F 3 "~" H 13250 5200 50  0001 C CNN
+	1    13250 5200
 	0    1    1    0
 $EndComp
@@
 L power:+BATT #PWR0109
 U 1 1 5D67BC2E
-P 15300 7650
-F 0 "#PWR0109" H 15300 7500 50  0001 C CNN
-F 1 "+BATT" H 15400 7800 50  0000 C CNN
-F 2 "" H 15300 7650 50  0001 C CNN
-F 3 "" H 15300 7650 50  0001 C CNN
-	1    15300 7650
+P 13250 5000
+F 0 "#PWR0109" H 13250 4850 50  0001 C CNN
+F 1 "+BATT" H 13350 5150 50  0000 C CNN
+F 2 "" H 13250 5000 50  0001 C CNN
+F 3 "" H 13250 5000 50  0001 C CNN
+	1    13250 5000
 	1    0    0    -1
 $EndComp
@@
 L power:GND #PWR0117
 U 1 1 5D67BC75
-P 14950 7800
-F 0 "#PWR0117" H 14950 7550 50  0001 C CNN
-F 1 "GND" H 14955 7627 50  0000 C CNN
-F 2 "" H 14950 7800 50  0001 C CNN
-F 3 "" H 14950 7800 50  0001 C CNN
-	1    14950 7800
-	1    0    0    -1
-$EndComp
-Wire Wire Line
-	15200 7650 14950 7650
-Wire Wire Line
-	14950 7650 14950 7800
+P 12900 5150
+F 0 "#PWR0117" H 12900 4900 50  0001 C CNN
+F 1 "GND" H 12905 4977 50  0000 C CNN
+F 2 "" H 12900 5150 50  0001 C CNN
+F 3 "" H 12900 5150 50  0001 C CNN
+	1    12900 5150
+	1    0    0    -1
+$EndComp
+Wire Wire Line
+	13150 5000 12900 5000
+Wire Wire Line
+	12900 5000 12900 5150
 Text GLabel 10500 3300 2    50   Input ~ 0
 BAT_MON
@@
 Text GLabel 10500 3200 2    50   Input ~ 0
 ACC_INT
-Wire Wire Line
-	10900 3600 10900 3700
-Connection ~ 10900 3700
 Text GLabel 12750 3150 0    50   Input ~ 0
 CS
@@
 NoConn ~ 9300 2800
 NoConn ~ 9300 3000
+Wire Wire Line
+	12200 4450 12200 4650
+Wire Wire Line
+	10900 5700 10900 5900
+Connection ~ 10900 5900
+Wire Wire Line
+	10900 5900 10900 6000
+Wire Wire Line
+	10900 6000 10900 6300
+Wire Wire Line
+	10900 6300 9900 6300
+Connection ~ 10900 6000
+Connection ~ 9900 6300
 $EndSCHEMATC
